File: 01_hardware/pcb/pcb.kicad_sch (KiCad schematic)
At the start: 4 parts, among them J1 Conn_01x03_Socket

Commit message: Text
Other:
- title: Pflanzensensor V1.0 -> Pflanzensensor
Changed lines of the file:
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@@
 	(paper "A5")
 	(title_block
-		(title "Pflanzensensor V1.0")
+		(title "Pflanzensensor")
+		(date "2026-03-18")
+		(rev "1.0")
 	)
 	(wire
